Commit message: third commit

File: src/my_robot/urdf/my_robot.xacro (robot description, xacro)
@@ -1,9 +1,10 @@
 <?xml version='1.0'?>
 <robot name="my_robot" xmlns:xacro="http://www.ros.org/wiki/xacro">
+<xacro:include filename="$(find my_robot)/urdf/my_robot.gazebo" />
   <link name="left_wheel">
     <visual name="left_wheel_visual">
       <origin xyz="0 0 0" rpy="0 1.5707 1.5707"/>
       <geometry>
-        <cylinder radius="0.1" lenght="0.05"/>
+        <cylinder radius="0.1" length="0.05"/>
       </geometry>
     </visual>
@@ -11,5 +12,5 @@
       <origin xyz="0 0 0" rpy="0 1.5707 1.5707"/>
       <geometry>
-        <cylinder radius="0.1" lenght="0.05"/>
+        <cylinder radius="0.1" length="0.05"/>
       </geometry>
     </collision>
@@ -45,5 +46,5 @@
       <origin xyz="0 0 0" rpy="0 1.5707 1.5707"/>
       <geometry>
-        <cylinder radius="0.1" lenght="0.05"/>
+        <cylinder radius="0.1" length="0.05"/>
       </geometry>
     </visual>
@@ -51,5 +52,5 @@
       <origin xyz="0 0 0" rpy="0 1.5707 1.5707"/>
       <geometry>
-        <cylinder radius="0.1" lenght="0.05"/>
+        <cylinder radius="0.1" length="0.05"/>
       </geometry>
     </collision>
@@ -117,3 +118,73 @@
     </visual>
   </link>
+<link name="camera">
+    <visual name="camera_visual">
+      <origin xyz="0 0 0" rpy="0 0 0"/>
+      <geometry>
+        <box size=".05 .05 .05"/>
+      </geometry>
+    </visual>
+    <collision name='camera_collision'>
+      <origin xyz="0 0 0" rpy="0 0 0"/>
+      <geometry>
+        <box size=".05 .05 .05"/>
+      </geometry>
+    </collision>
+    <inertial name='box_inertia'>
+      <mass value="0.1"/>
+      <origin xyz="0.0 0 0" rpy="0 0 0"/>
+        <inertia
+          ixx="1e-6" ixy="0" ixz="0"
+          iyy="1e-6" iyz="0"
+          izz="1e-6"
+      />
+    </inertial>
+   </link>
+  <joint type="fixed"  name="camera_joint">
+    <origin xyz="0.2 0 0" rpy="0 0 0" />
+      <child link="camera"/>
+    <parent link="chassis"/>
+    <axis xyz="0 1 0" rpy="0 0 0"/>
+   </joint>
+<link name="hokuyo">
+    <visual name="lidar_visual">
+      <origin xyz="0 0 0" rpy="0 0 0"/>
+      <geometry>
+        <mesh filename="package://my_robot/meshes/hokuyo.dae"/>
+      </geometry>
+    </visual>
+    <collision name='lidar_collision'>
+      <origin xyz="0 0 0" rpy="0 0 0"/>
+      <geometry>
+        <box size=".1 .1 .1"/>
+      </geometry>
+    </collision>
+    <inertial name='lidar_inertia'>
+      <mass value="1e-5"/>
+      <origin xyz="0.0 0 0" rpy="0 0 0"/>
+        <inertia
+          ixx="1e-6" ixy="0" ixz="0"
+          iyy="1e-6" iyz="0"
+          izz="1e-6"
+      />
+    </inertial>
+   </link>
+  <joint type="fixed"  name="hokuyo_joint">
+    <origin xyz="0.15 0 0.1" rpy="0 0 0" />
+      <child link="hokuyo"/>
+    <parent link="chassis"/>
+    <axis xyz="0 1 0" rpy="0 0 0"/>
+   </joint>
+<gazebo reference="left_wheel">
+    <material>Gazebo/Green</material>
+</gazebo>
+<gazebo reference="right_wheel">
+    <material>Gazebo/Green</material>
+</gazebo>
+<gazebo reference="chassis">
+    <material>Gazebo/Blue</material>
+</gazebo>
+<gazebo reference="camera">
+    <material>Gazebo/Red</material>
+</gazebo>
 </robot>
